Commit message: 第二十次提交：完成moveit2和上位机、下位机的连接代码编写加虚拟测试。接下来进行真机测试

File: src/rm_algorithm/armbot_moveit2/config/rm_description.ros2_control.xacro (robot description, xacro)
@@ -6,61 +6,47 @@
             <hardware>
                 <!-- By default, set up controllers for simulation. This won't work on real hardware -->
-                <plugin>mock_components/GenericSystem</plugin>
+                <plugin>arm_hardware/ArmHardwareInterface</plugin>
             </hardware>
             <joint name="joint1">
                 <command_interface name="position"/>
                 <state_interface name="position">
-                  <param name="initial_value">${initial_positions['joint1']}</param>
+                  <param name="initial_value">0.0</param>
                 </state_interface>
-                <state_interface name="velocity"/>
             </joint>
             <joint name="joint2">
                 <command_interface name="position"/>
                 <state_interface name="position">
-                  <param name="initial_value">${initial_positions['joint2']}</param>
+                  <param name="initial_value">0.0</param>
                 </state_interface>
-                <state_interface name="velocity"/>
             </joint>
             <joint name="joint3">
                 <command_interface name="position"/>
                 <state_interface name="position">
-                  <param name="initial_value">${initial_positions['joint3']}</param>
+                  <param name="initial_value">0.0</param>
                 </state_interface>
-                <state_interface name="velocity"/>
             </joint>
             <joint name="joint4">
                 <command_interface name="position"/>
                 <state_interface name="position">
-                  <param name="initial_value">${initial_positions['joint4']}</param>
+                  <param name="initial_value">0.0</param>
                 </state_interface>
-                <state_interface name="velocity"/>
             </joint>
             <joint name="joint5">
                 <command_interface name="position"/>
                 <state_interface name="position">
-                  <param name="initial_value">${initial_positions['joint5']}</param>
+                  <param name="initial_value">0.0</param>
                 </state_interface>
-                <state_interface name="velocity"/>
             </joint>
             <joint name="joint6">
                 <command_interface name="position"/>
                 <state_interface name="position">
-                  <param name="initial_value">${initial_positions['joint6']}</param>
+                  <param name="initial_value">0.0</param>
                 </state_interface>
-                <state_interface name="velocity"/>
             </joint>
             <joint name="joint_gripper_left">
                 <command_interface name="position"/>
                 <state_interface name="position">
-                  <param name="initial_value">${initial_positions['joint_gripper_left']}</param>
+                  <param name="initial_value">0.0</param>
                 </state_interface>
-                <state_interface name="velocity"/>
-            </joint>
-            <joint name="joint_gripper_right">
-                <command_interface name="position"/>
-                <state_interface name="position">
-                  <param name="initial_value">${initial_positions['joint_gripper_right']}</param>
-                </state_interface>
-                <state_interface name="velocity"/>
             </joint>
         </ros2_control>

File: src/rm_description/urdf/mechine_arm.urdf (robot description, URDF)
Before this commit: robot rm_description, 13 links, 12 joints
Joints:
- joint joint_gripper_right: axis 0 0 -1 -> 0 0 1; mimic (none) -> joint=joint_gripper_left
