Commit message: 第二十一次提交：完成上车电机方向测试（1.0版本）

File: src/rm_description/urdf/mechine_arm.urdf (robot description, URDF)
Before this commit: robot rm_description, 13 links, 12 joints
Joints:
- joint joint_gripper_left: limit lower=0.0 upper=0.06 effort=1000 velocity=1.0 -> lower=0.0 upper=0.06 effort=10 velocity=1.0
- joint joint_gripper_right: limit lower=-0.06 upper=0.0 effort=1000 velocity=1.0 -> lower=-0.06 upper=0.0 effort=10 velocity=1.0
