Commit message: 使用 Git LFS 管理大文件

File: src/rm_description/urdf/engineer.urdf (robot description, URDF)
Before this commit: robot engineer, 7 links, 6 joints
Links:
- added link base_footprint; visual box size=0.1 0.1 0.01
- added link livox_frame, mass 0.17859; collision mesh filename=package://rm_description/meshes/radar.STL; visual mesh filename=package://rm_description/meshes/radar.STL
Joints:
- added joint joint_base_footprint: type fixed, parent base_footprint, child base_link, origin xyz=0 0 0.18113 rpy=0 0 0
- added joint livox_frame_joint: type fixed, parent base_link, child livox_frame, origin xyz=0.1572 -0.1665 0.0922 rpy=0 0 0
