Commit message: 第四十次提交：生成ikfast求解器，将其加载到moveit2中

File: src/rm_algorithm/engineer_moveit2/config/engineer.ros2_control.xacro (robot description, xacro)
@@ -5,6 +5,6 @@
         <ros2_control name="${name}" type="system">
             <hardware>
-                <plugin>arm_hardware/ArmHardwareInterface</plugin>
-                <!-- <plugin>mock_components/GenericSystem</plugin> -->
+                <!-- <plugin>arm_hardware/ArmHardwareInterface</plugin> -->
+                <plugin>mock_components/GenericSystem</plugin>
             </hardware>
             <joint name="joint_1">

File: src/rm_description/urdf/arm.xacro (robot description, xacro)
@@ -211,5 +211,5 @@
       <child link="link_5" />
       <axis xyz="0 0 -1" />
-      <limit lower="-1.57" upper="1.57" effort="10" velocity="3" />
+      <limit lower="-1.8" upper="1.8" effort="10" velocity="3" />
     </joint>
     <!-- link_6 -->
